File: bandara_ckt_pcb_naveen.kicad_pcb (KiCad board)
At the start: 2 copper layers, 98.8 x 81.1 mm, 54 parts, among them J1 Nanopore, U1 MCP4725xxx-xCH, U2 ADS1115IDGS, U3 AD820, U4 Dual Power Supply, U5 AD820, U6 AD820

Commit message: Final commit after changing C2 footprint
Parts:
- C2: footprint Capacitor_Tantalum_SMD:CP_EIA-1608-08_AVX-J_Pad1.25x1.05mm_HandSolder -> Capacitor_Tantalum_SMD:CP_EIA-3216-10_Kemet-I
- moved TP4 1.50 mm to (84.2, 51.7)
Routing:
- net GND: track 386.6 -> 388.8 mm
- net +5V: track 239.3 -> 240.8 mm
- net +3.3V: track 35.7 -> 36.7 mm
- net Net-(U1-VOUT): track 101.8 -> 102.5 mm
