File: bandara_ckt_pcb_naveen.kicad_sch (KiCad schematic)
At the start: 49 parts, among them J1 Nanopore, U1 MCP4725xxx-xCH, U2 ADS1115IDGS, U3 AD820, U4 Dual Power Supply, U5 AD820, U6 AD820

Commit message: Review version of Bandara circuit
Parts:
- added R14: 1M, Resistor_SMD:R_0603_1608Metric_Pad0.98x0.95mm_HandSolder, symbol Device:R
Connections:
- net at R13.2, TP15.1, U6.6 (Vout): now also R14.2
- net at R10.2, U6.2 (-IN): now also R14.1
Changed lines of the file:
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@@
 	)
 	(junction
+		(at 231.14 90.17)
+		(diameter 0)
+		(color 0 0 0 0)
+	)
+	(junction
 		(at 148.59 53.34)
 		(diameter 0)
@@
 	)
 	(junction
+		(at 259.08 95.25)
+		(diameter 0)
+		(color 0 0 0 0)
+	)
+	(junction
 		(at 109.22 132.08)
 		(diameter 0)
@@
 	(wire
 		(pts
-			(xy 227.33 95.25) (xy 233.68 95.25)
+			(xy 229.87 95.25) (xy 233.68 95.25)
 		)
 		(stroke
@@
 	(wire
 		(pts
-			(xy 227.33 95.25) (xy 227.33 119.38)
+			(xy 229.87 95.25) (xy 229.87 97.79)
 		)
 		(stroke
@@
 	(wire
 		(pts
+			(xy 259.08 95.25) (xy 265.43 95.25)
+		)
+		(stroke
+			(width 0)
+			(type default)
+		)
+	)
+	(wire
+		(pts
 			(xy 227.33 133.35) (xy 233.68 133.35)
 		)
@@
 	(wire
 		(pts
-			(xy 229.87 90.17) (xy 233.68 90.17)
+			(xy 229.87 90.17) (xy 231.14 90.17)
 		)
 		(stroke
@@
 	(wire
 		(pts
-			(xy 256.54 95.25) (xy 265.43 95.25)
+			(xy 256.54 95.25) (xy 259.08 95.25)
 		)
 		(stroke
@@
 	(wire
 		(pts
+			(xy 259.08 121.92) (xy 259.08 95.25)
+		)
+		(stroke
+			(width 0)
+			(type default)
+		)
+	)
+	(wire
+		(pts
 			(xy 115.57 133.35) (xy 115.57 139.7)
 		)
@@
 	(wire
 		(pts
-			(xy 105.41 85.09) (xy 111.76 85.09)
+			(xy 226.06 121.92) (xy 226.06 93.98)
 		)
 		(stroke
@@
 	(wire
 		(pts
+			(xy 105.41 85.09) (xy 111.76 85.09)
+		)
+		(stroke
+			(width 0)
+			(type default)
+		)
+	)
+	(wire
+		(pts
 			(xy 68.58 58.42) (xy 80.01 58.42)
 		)
@@
 	(wire
 		(pts
+			(xy 252.73 121.92) (xy 259.08 121.92)
+		)
+		(stroke
+			(width 0)
+			(type default)
+		)
+	)
+	(wire
+		(pts
 			(xy 168.91 53.34) (xy 172.72 53.34)
 		)
@@
 	(wire
 		(pts
-			(xy 111.76 74.93) (xy 111.76 76.2)
+			(xy 111.76 72.39) (xy 111.76 76.2)
 		)
 		(stroke
@@
 	(wire
 		(pts
+			(xy 226.06 93.98) (xy 231.14 93.98)
+		)
+		(stroke
+			(width 0)
+			(type default)
+		)
+	)
+	(wire
+		(pts
 			(xy 134.62 154.94) (xy 238.76 154.94)
 		)
@@
 	(wire
 		(pts
+			(xy 231.14 93.98) (xy 231.14 90.17)
+		)
+		(stroke
+			(width 0)
+			(type default)
+		)
+	)
+	(wire
+		(pts
 			(xy 62.23 132.08) (xy 62.23 137.16)
 		)
@@
 	(wire
 		(pts
+			(xy 245.11 121.92) (xy 226.06 121.92)
+		)
+		(stroke
+			(width 0)
+			(type default)
+		)
+	)
+	(wire
+		(pts
 			(xy 31.75 124.46) (xy 34.29 124.46)
 		)
@@
 	(wire
 		(pts
+			(xy 231.14 90.17) (xy 233.68 90.17)
+		)
+		(stroke
+			(width 0)
+			(type default)
+		)
+	)
+	(wire
+		(pts
 			(xy 59.69 57.15) (xy 59.69 60.96)
 		)
@@
 	(symbol
 		(lib_id "power:GND")
-		(at 111.76 74.93 180)
+		(at 111.76 72.39 180)
 		(unit 1)
 		(exclude_from_sim no)
@@
 		(dnp no)
 		(property "Reference" "#PWR017"
-			(at 111.76 68.58 0)
+			(at 111.76 66.04 0)
 			(effects
 				(font
@@
 		)
 		(property "Value" "GND"
-			(at 115.062 74.422 0)
+			(at 115.062 71.882 0)
 			(effects
 				(font
@@
 		)
 		(property "Footprint" ""
-			(at 111.76 74.93 0)
+			(at 111.76 72.39 0)
 			(effects
 				(font
@@
 		)
 		(property "Datasheet" ""
-			(at 111.76 74.93 0)
+			(at 111.76 72.39 0)
 			(effects
 				(font
@@
 		)
 		(property "Description" "Power symbol creates a global label with name \"GND\" , ground"
-			(at 111.76 74.93 0)
+			(at 111.76 72.39 0)
 			(effects
 				(font
@@
 	(symbol
 		(lib_id "power:GND")
-		(at 227.33 119.38 0)
+		(at 229.87 97.79 0)
 		(unit 1)
 		(exclude_from_sim no)
@@
 		(on_board yes)
 		(dnp no)
-		(fields_autoplaced yes)
 		(property "Reference" "#PWR032"
-			(at 227.33 125.73 0)
+			(at 229.87 104.14 0)
 			(effects
 				(font
@@
 		)
 		(property "Value" "GND"
-			(at 227.33 124.46 0)
+			(at 230.378 101.854 0)
 			(effects
 				(font
@@
 		)
 		(property "Footprint" ""
-			(at 227.33 119.38 0)
+			(at 229.87 97.79 0)
 			(effects
 				(font
@@
 		)
 		(property "Datasheet" ""
-			(at 227.33 119.38 0)
+			(at 229.87 97.79 0)
 			(effects
 				(font
@@
 		)
 		(property "Description" "Power symbol creates a global label with name \"GND\" , ground"
-			(at 227.33 119.38 0)
+			(at 229.87 97.79 0)
 			(effects
 				(font
@@
 		)
 		(property "Value" "TestPoint"
-			(at 221.996 93.218 0)
+			(at 219.202 103.886 90)
 			(effects
 				(font
@@
 					(unit 1)
 				)
+			)
+		)
+	)
+	(symbol
+		(lib_id "Device:R")
+		(at 248.92 121.92 90)
+		(unit 1)
+		(exclude_from_sim no)
+		(in_bom yes)
+		(on_board yes)
+		(dnp no)
+		(property "Reference" "R14"
+			(at 248.92 116.84 90)
+			(effects
+				(font
+					(size 1.27 1.27)
+				)
+			)
+		)
+		(property "Value" "1M"
+			(at 248.92 119.126 90)
+			(effects
+				(font
+					(size 1.27 1.27)
+				)
+			)
+		)
+		(property "Footprint" "Resistor_SMD:R_0603_1608Metric_Pad0.98x0.95mm_HandSolder"
+			(at 248.92 123.698 90)
+			(effects
+				(font
+					(size 1.27 1.27)
+				)
+				(hide yes)
+			)
+		)
+		(property "Datasheet" "~"
+			(at 248.92 121.92 0)
+			(effects
+				(font
+					(size 1.27 1.27)
+				)
+				(hide yes)
+			)
+		)
+		(property "Description" "Resistor"
+			(at 248.92 121.92 0)
+			(effects
+				(font
+					(size 1.27 1.27)
+				)
+				(hide yes)
+			)
+		)
+		(pin "2"
+		)
+		(pin "1"
+		)
+		(instances
+			(project ""
+				(path "/3ad0222e-ebc6-46e3-b177-fd821a5b6ee2"
+					(reference "R14")
+					(unit 1)
+				)

Commit message: PCB and Schematic updated after YES from Bandara
Parts:
- added C2: 10u, Capacitor_Tantalum_SMD:CP_EIA-1608-08_AVX-J_Pad1.25x1.05mm_HandSolder, symbol Device:C
- added C3: 100n, Capacitor_SMD:C_0805_2012Metric_Pad1.18x1.45mm_HandSolder, symbol Device:C
- added TP12, TP3: TestPoint, TestPoint:TestPoint_THTPad_D2.0mm_Drill1.0mm, symbol Connector:TestPoint
- TP1, TP16, TP2, TP5, TP6: footprint TestPoint:TestPoint_THTPad_1.5x1.5mm_Drill0.7mm -> TestPoint:TestPoint_THTPad_D2.0mm_Drill1.0mm
- TP10: renamed from TP9; footprint TestPoint:TestPoint_THTPad_1.5x1.5mm_Drill0.7mm -> TestPoint:TestPoint_THTPad_D2.0mm_Drill1.0mm
- TP11: renamed from TP10; footprint TestPoint:TestPoint_THTPad_1.5x1.5mm_Drill0.7mm -> TestPoint:TestPoint_THTPad_D2.0mm_Drill1.0mm
- TP13: renamed from TP11; footprint TestPoint:TestPoint_THTPad_1.5x1.5mm_Drill0.7mm -> TestPoint:TestPoint_THTPad_D2.0mm_Drill1.0mm
- TP14: renamed from TP12; footprint TestPoint:TestPoint_THTPad_1.5x1.5mm_Drill0.7mm -> TestPoint:TestPoint_THTPad_D2.0mm_Drill1.0mm
- TP15: renamed from TP13; footprint TestPoint:TestPoint_THTPad_1.5x1.5mm_Drill0.7mm -> TestPoint:TestPoint_THTPad_D2.0mm_Drill1.0mm
- TP17: renamed from TP14; footprint TestPoint:TestPoint_THTPad_1.5x1.5mm_Drill0.7mm -> TestPoint:TestPoint_THTPad_D2.0mm_Drill1.0mm
- TP18: renamed from TP15; footprint TestPoint:TestPoint_THTPad_1.5x1.5mm_Drill0.7mm -> TestPoint:TestPoint_THTPad_D2.0mm_Drill1.0mm
- TP4: renamed from TP3; footprint TestPoint:TestPoint_THTPad_1.5x1.5mm_Drill0.7mm -> TestPoint:TestPoint_THTPad_D2.0mm_Drill1.0mm
- TP7: renamed from TP4; footprint TestPoint:TestPoint_THTPad_1.5x1.5mm_Drill0.7mm -> TestPoint:TestPoint_THTPad_D2.0mm_Drill1.0mm
- TP8: renamed from TP7; footprint TestPoint:TestPoint_THTPad_1.5x1.5mm_Drill0.7mm -> TestPoint:TestPoint_THTPad_D2.0mm_Drill1.0mm
- TP9: renamed from TP8; footprint TestPoint:TestPoint_THTPad_1.5x1.5mm_Drill0.7mm -> TestPoint:TestPoint_THTPad_D2.0mm_Drill1.0mm
- renumbered C8 to C10, C9 to C11, C10 to C12, C11 to C13, C12 to C14, C2 to C4, C3 to C5, C4 to C6, C5 to C7, C6 to C8, C7 to C9, R14 to R12, R12 to R13, R13 to R14
Connections:
- net +5V: no longer U1.3 (VDD)
- net GND: now also C2.2, C3.2
- net at C9.1, J1.2 (Pin_2), R8.1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: now also TP12.1
- net +3.3V: now reaches A1.4 (3V3)
- net +3.3V: now also U1.3 (VDD), C2.1, C3.1, TP3.1
- no-connect marks 24 -> 23
Other:
- moved on the sheet: TP1, TP2

Commit message: Final commit after changing C2 footprint
Parts:
- C2: footprint Capacitor_Tantalum_SMD:CP_EIA-1608-08_AVX-J_Pad1.25x1.05mm_HandSolder -> Capacitor_Tantalum_SMD:CP_EIA-3216-10_Kemet-I
Changed lines of the file:
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@@
 			)
 		)
-		(property "Footprint" "Capacitor_Tantalum_SMD:CP_EIA-1608-08_AVX-J_Pad1.25x1.05mm_HandSolder"
+		(property "Footprint" "Capacitor_Tantalum_SMD:CP_EIA-3216-10_Kemet-I"
 			(at 95.25 53.6448 0)
 			(effects
